File: aircraft.kicad_sch (KiCad schematic)
At the start: 0 parts

Commit message: power supply and navigation unit
Other:
- company: (none) -> Breno Soares Alves
- title: (none) -> Gravitum Flight Control System
Changed lines of the file:
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@@
 	(generator_version "9.0")
 	(paper "A4")
+	(title_block
+		(title "Gravitum Flight Control System")
+		(company "Breno Soares Alves")
+	)
 	(sheet
 		(at 152.4 43.18)
@@
 			(project "aircraft"
 				(path "/8dc22ddc-eb0a-4b80-a714-26a959e826d2"
-					(page "4")
+					(page "5")
 				)
 			)
@@
 			(project "aircraft"
 				(path "/8dc22ddc-eb0a-4b80-a714-26a959e826d2"
-					(page "5")
-				)
-			)
+					(page "4")
+				)
+			)
