File: navigation_unit.kicad_sch (KiCad schematic)
At the start: 1 part, among them U4 STM32F405RGT6

Commit message: power supply and navigation unit
Parts:
- added C12, C14, C15, C16, C17, C18, C19, C20, C21, C22, C25, C29: 100n, symbol Device:C
- added C13: 10u, symbol Device:C_Polarized
- added C23, C24: 2u2, symbol Device:C
- added C26: 1u, symbol Device:C_Polarized
- added C27, C28: 10p, symbol Device:C
- added D3: B, symbol Device:LED
- added D4: Y, symbol Device:LED
- added D5: R, symbol Device:LED
- added D6: G, symbol Device:LED
- added FB1: FerriteBead, symbol Device:FerriteBead
- added R10, R11, R12, R9: 560, symbol Device:R
- added R13, R14: 10k, symbol Device:R
- added R15, R16, R17, R18: 4k7, symbol Device:R
- added R8: 620, symbol Device:R
- added S1: SKRPACE010, SKRPACE010:SW_SKRPACE010, symbol Aircraft_Components:SKRPACE010
- added U13, U14: TDD01H0SB1R, SOT_TDDSB1R_CNK, symbol Aircraft_Components:TDD01H0SB1R
- added Y1: 25MHz, symbol Device:Crystal_GND24
Connections:
- net +3.3V: now reaches U4.1 (VBAT)
- net +3.3V: now also U4.19 (VDD), U4.32 (VDD__1), U4.48 (VDD__2), U4.64 (VDD__3), C12.1, C13.1, C14.1, C15.1, C16.1, C17.1, C18.1, C19.1, C20.1, C21.1, C22.1, FB1.1, R15.2, R16.2, R17.2, R18.2, U13.1, U14.1
- net GND: now reaches U4.12 (VSSA)
- net GND: now also U4.18 (VSS), U4.63 (VSS__1), C12.2, C13.2, C14.2, C15.2, C16.2, C17.2, C18.2, C19.2, C20.2, C21.2, C22.2, C23.2, C24.2, C25.2, C26.2, C27.2, C28.2, C29.2, R10.2, R11.2, R12.2, R9.2, S1.2, S1.4, U13.3, U14.3, Y1.2, Y1.4
- net NU_VDDA: now reaches U4.13 (VDDA)
- net NU_VDDA: now also C25.1, C26.1, FB1.2
- net NU_BOOT1: now reaches U4.28 (PB2/BOOT1)
- net NU_VCAP1: now reaches U4.31 (VCAP_1)
- net NU_VCAP1: now also C24.1
- net NU_VCAP2: now reaches U4.47 (VCAP_2)
- net NU_VCAP2: now also C23.1
- net NU_HSO_IN: now reaches U4.5 (PH0/OSC_IN)
- net NU_HSO_IN: now also C27.1, Y1.1
- net NU_HSO_OUT: now reaches U4.6 (PH1/OSC_OUT)
- net NU_HSO_OUT: now also R8.1
- net NU_BOOT0: now reaches U4.60 (BOOT0)
- net NU_BOOT0: now also R13.1, R14.1
- net NU_NRST: now reaches U4.7 (NRST)
- net NU_NRST: now also C29.1, S1.1, S1.3
- new net: D4.1 (K), R11.1
- new net: C28.1, R8.2, Y1.3
- new net: R14.2, U14.2
- new net: D3.1 (K), R12.1
- new net: D6.1 (K), R9.1
- new net: R13.2, U13.2
- new net: D5.1 (K), R10.1
- new net LED_NU4: D3.2 (A)
- new net NU_I2C1_SCL: R16.1
- new net NU_I2C1_SDA: R15.1
- new net NU_I2C2_SCL: R18.1
- new net NU_I2C2_SDA: R17.1
- new net NU_LED1: D6.2 (A)
- new net NU_LED2: D5.2 (A)
- new net NU_LED3: D4.2 (A)
Other:
- note added: "2 capacitors per VDD pin"
- note added: "Boot Mode"
- note added: "Decoupling Capacitors"
- note added: "High Speed Oscilattor"
- note added: "I2C Pull up resistors"
- note added: "Navigation Unit"
- note added: "Reset button"
- note added: "Status LEDs"
- note added: "VCAP Filter"
- note added: "VDDA Filter"
- moved on the sheet: U4
