File: power_supply.kicad_sch (KiCad schematic)
At the start: 4 parts, among them J1 Conn_01x02_Pin, U1 INA226AIDGSR, U2 LD39200PU33R, U3 MIC26903YJL-TR

Commit message: power supply and navigation unit
Parts:
- added C1, C5, C6: 0.1u, symbol Device:C
- added C10, C11: 10u, symbol Device:C
- added C2: 2u2, symbol Device:C
- added C3, C4: 4u7, symbol Device:C
- added C7: 4n7, symbol Device:C
- added C8, C9: 100u, symbol Device:C
- added D1: D_Schottky, symbol Device:D_Schottky
- added D2: G, symbol Device:LED
- added L1: 15u, symbol Device:L
- added R1: 2m, symbol Device:R
- added R2, R3: 10k, symbol Device:R
- added R4: 19k6, symbol Device:R
- added R5: 6k8, symbol Device:R
- added R6: 1k3, symbol Device:R
- added R7: 560, symbol Device:R
Connections:
- net VIN is gone; now on net VCC: J1.1 (Pin_1)
- net GND: now also U1.1 (A1), U1.2 (A0), U1.7 (GND), U1.8 (VBUS), U1.9 (VIN-), U2.3 (GND), U2.7 (GND), U3.13 (PVIN), U3.14 (PVIN), U3.15 (PVIN), U3.16 (PVIN), U3.17 (PVIN), U3.18 (PVIN), U3.19 (PVIN), U3.2 (PGND), U3.21 (PGND), U3.23 (SGND), U3.27 (VIN), U3.29 (EPAD), U3.5 (PGND), U3.6 (PGND), U3.7 (PGND), U3.8 (PGND), C1.1, C10.1, C11.2, C2.1, C3.1, C3.2, C4.1, C4.2, C8.2, C9.2, D2.1 (K), R1.1, R2.1, R6.2
- net at U3.1 (PVDD): now also C2.2
- net PS_CS: now reaches U3.10 (SW)
- net PS_CS: now also U3.11 (SW), U3.12 (SW), U3.22 (CS), U3.4 (SW), U3.9 (SW), C5.1, C6.1, L1.1
- net PS_BST: now reaches U3.20 (BST)
- net PS_BST: now also C5.2, D1.1 (K)
- net PS_FB: now reaches U3.24 (FB)
- net PS_FB: now also C7.2, R4.1, R5.2, R6.1
- net PS_PG: now reaches U3.25 (PG)
- net PS_PG: now also R3.1
- net PS_EN: now reaches U3.26 (EN)
- net PS_EN: now also R2.2
- net at U3.28 (VDD): now also D1.2 (A), R3.2
- net VCC: now reaches U1.10 (VIN+)
- net VCC: now also R1.2
- net I2C_INA_SDA: now reaches U1.4 (SDA)
- net I2C_INA_SCL: now reaches U1.5 (SCL)
- net +5V: now reaches U1.6 (VS)
- net +5V: now also U2.5 (EN), U2.6 (IN), C1.2, C10.2, C7.1, C8.1, C9.1, L1.2, R5.1, R7.2
- net +3.3V: now reaches U2.1 (OUT)
- net +3.3V: now also U2.2 (ADJ/SENSE), C11.1
- new net: D2.2 (A), R7.1
- new net: C6.2, R4.2
- no-connect marks 0 -> 2
Other:
- note added: "3.3V Linear Converter"
- note added: "5V Bulk Converter"
- note added: "Battery Entry"
- note added: "I2C Address: 0x40"
- note added: "Power Monitoring"
- note added: "REVIEW: Verify if ALERT Pin is required"
- note added: "Shunt"
- company: (none) -> Breno Soares Alves
- title: (none) -> Power Supply
- moved on the sheet: U1, U2, U3
