File: Hardware/other_connections.kicad_sch (KiCad schematic)
At the start: 45 parts, among them J12 Conn_02x05_Odd_Even, J13 Conn_01x02, J14 USB_B_Micro, J15 Conn_02x05_Odd_Even, J16 USB_B_Micro, J17 USB_B_Micro, J18 USB_B_Micro, U16 CH330N, U17 CH330N

Commit message: hardware version 0.1.2, minor improvements and footprint selection (missing some gnss and bulk regulator components
Parts:
- J12, J15: footprint (none) -> Aircraft_Footprints:JST_PHD_B10B-PHDSS_2x05_P2.00mm_Vertical
- J13: footprint (none) -> Connector_JST:JST_PH_S2B-PH-K_1x02_P2.00mm_Horizontal
- J14, J16, J17, J18: footprint (none) -> Connector_USB:USB_Micro-B_Molex_47346-0001
- JP2: footprint (none) -> Jumper:SolderJumper-3_P1.3mm_Open_RoundedPad1.0x1.5mm_NumberLabels
- JP3, JP4: footprint (none) -> Jumper:SolderJumper-2_P1.3mm_Open_RoundedPad1.0x1.5mm
Changed lines of the file:
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@@
 	(title_block
 		(title "Other Connections")
-		(rev "0.1.1")
+		(rev "0.1.2")
 		(company "Breno Soares Alves")
 	)
@@
 			)
 		)
-		(property "Footprint" ""
+		(property "Footprint" "Aircraft_Footprints:JST_PHD_B10B-PHDSS_2x05_P2.00mm_Vertical"
 			(at 146.05 154.94 0)
 			(effects
@@
 			)
 		)
-		(property "Footprint" ""
+		(property "Footprint" "Connector_USB:USB_Micro-B_Molex_47346-0001"
 			(at 215.9 46.99 0)
 			(effects
@@
 			)
 		)
-		(property "Footprint" ""
+		(property "Footprint" "Jumper:SolderJumper-3_P1.3mm_Open_RoundedPad1.0x1.5mm_NumberLabels"
 			(at 105.41 96.52 0)
 			(effects
@@
 			)
 		)
-		(property "Footprint" ""
+		(property "Footprint" "Connector_JST:JST_PH_S2B-PH-K_1x02_P2.00mm_Horizontal"
 			(at 113.03 106.68 0)
 			(effects
@@
 			)
 		)
-		(property "Footprint" ""
+		(property "Footprint" "Aircraft_Footprints:JST_PHD_B10B-PHDSS_2x05_P2.00mm_Vertical"
 			(at 107.95 154.94 0)
 			(effects
@@
 			)
 		)
-		(property "Footprint" ""
+		(property "Footprint" "Jumper:SolderJumper-2_P1.3mm_Open_RoundedPad1.0x1.5mm"
 			(at 168.91 88.9 0)
 			(effects
@@
 			)
 		)
-		(property "Footprint" ""
+		(property "Footprint" "Connector_USB:USB_Micro-B_Molex_47346-0001"
 			(at 224.79 105.41 0)
 			(effects
@@
 			)
 		)
-		(property "Footprint" ""
+		(property "Footprint" "Connector_USB:USB_Micro-B_Molex_47346-0001"
 			(at 142.24 48.26 0)
 			(effects
@@
 			)
 		)
-		(property "Footprint" ""
+		(property "Footprint" "Jumper:SolderJumper-2_P1.3mm_Open_RoundedPad1.0x1.5mm"
 			(at 238.76 88.9 0)
 			(effects
@@
 			)
 		)
-		(property "Footprint" ""
+		(property "Footprint" "Connector_USB:USB_Micro-B_Molex_47346-0001"
 			(at 153.67 105.41 0)
 			(effects

Commit message: board placement, no trails, just pain
Parts:
- removed R45: 10, Resistor_SMD:R_0603_1608Metric, symbol Device:R
- C60, C61, C62, C63: Digikey_Link (none) -> https://www.digikey.com.br/pt/products/detail/kemet/C0603C1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; MPN (none) -> C0603C104K8RACTU
- D12, D13, D15, D16: Digikey_Link (none) -> https://www.digikey.com.br/pt/products/detail/evvo/sd103aws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; MPN (none) -> SD103AWS
- D14, D17: footprint LED_SMD:LED_0603_1608Metric -> LED_SMD:LED_0603_1608Metric_Pad1.05x0.95mm_HandSolder; Digikey_Link (none) -> https://www.digikey.com.br/pt/products/detail/liteon/LTST-S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; MPN (none) -> LTST-S270KGKT
- FB3, FB4, FB5, FB6: footprint Inductor_SMD:L_0805_2012Metric -> Inductor_SMD:L_0805_2012Metric_Pad1.05x1.20mm_HandSolder; Digikey_Link (none) -> https://www.digikey.com.br/pt/products/detail/laird-signal-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; MPN (none) -> HZ0805E601R-10
- J12, J15: Digikey_Link (none) -> https://www.digikey.com.br/pt/products/detail/jst-sales-ame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; MPN (none) -> B10B-PHDSS
- J13: Digikey_Link (none) -> https://www.digikey.com.br/pt/products/detail/jst-sales-ame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; MPN (none) -> S2B-PH-K-S
- J14, J16, J17, J18: Digikey_Link (none) -> https://www.digikey.com.br/pt/products/detail/molex/0473461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; MPN (none) -> 0473461001
- R35, R36: footprint Resistor_SMD:R_0603_1608Metric_Pad0.98x0.95mm_HandSolder -> Resistor_SMD:R_0402_1005Metric_Pad0.72x0.64mm_HandSolder; Digikey_Link (none) -> https://www.digikey.com.br/pt/products/detail/yageo/RC0603J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; MPN (none) -> RC0603JR-070RL
- R37, R38, R39, R40, R41, R42, R43, R44: footprint Resistor_SMD:R_0603_1608Metric -> Resistor_SMD:R_0402_1005Metric_Pad0.72x0.64mm_HandSolder; Digikey_Link (none) -> https://www.digikey.com.br/pt/products/detail/stackpole-ele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; MPN (none) -> RMCF0603FT10R0
- R46, R47, R50, R51: footprint Resistor_SMD:R_0603_1608Metric -> Resistor_SMD:R_0603_1608Metric_Pad0.98x0.95mm_HandSolder; Digikey_Link (none) -> https://www.digikey.com.br/pt/products/detail/yageo/RC0603F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; MPN (none) -> RC0603FR-0722RL
- R48, R52: footprint Resistor_SMD:R_0603_1608Metric -> Resistor_SMD:R_0603_1608Metric_Pad0.98x0.95mm_HandSolder; Digikey_Link (none) -> https://www.digikey.com.br/pt/products/detail/stackpole-ele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; MPN (none) -> RMCF0603FT560R
- R49, R53: Digikey_Link (none) -> https://www.digikey.com.br/pt/products/detail/stackpole-ele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; MPN (none) -> RMCF0603FT560R
- U16, U17: MPN (none) -> CH330N
Connections:
- net FCU_GPIOA renamed FCU_GPIO_A
- net FCU_GPIOB renamed FCU_GPIO_B
- net FCU_GPIOC renamed FCU_GPIO_C
- net FCU_GPIOD renamed FCU_GPIO_D
- net FCU_GPIOE renamed FCU_GPIO_E
- net FCU_GPIOF renamed FCU_GPIO_F
- net NU_GPIOA renamed NU_GPIO_A
- net NU_GPIOB renamed NU_GPIO_B
- net NU_GPIOC renamed NU_GPIO_C
- net NU_GPIOD renamed NU_GPIO_D
- net NU_GPIOE renamed NU_GPIO_E
- net NU_GPIOF renamed NU_GPIO_F
- net NU_I2C2_SCL renamed NU_I2C1_SCL
- net NU_I2C2_SDA renamed NU_I2C1_SDA
