File: Hardware/other_connections.kicad_sch (KiCad schematic)
At the start: 44 parts, among them J12 Conn_02x05_Odd_Even, J13 Conn_01x02, J14 USB_B_Micro, J15 Conn_02x05_Odd_Even, J16 USB_B_Micro, J17 USB_B_Micro, J18 USB_B_Micro, U16 CH330N, U17 CH330N

Commit message: hardware: better layout, no power supply and sensors
Connections:
- net FCU_USB_OTG_FS_DM renamed FCU_USB_OTG_FS_D-
- net FCU_USB_OTG_FS_DP renamed FCU_USB_OTG_FS_D+
Changed lines of the file:
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@@
 		)
 	)
-	(global_label "FCU_USB_OTG_FS_DP"
+	(global_label "FCU_USB_OTG_FS_D+"
 		(shape input)
 		(at 175.26 107.95 0)
@@
 		)
 		(property "Intersheetrefs" "${INTERSHEET_REFS}"
-			(at 198.0209 107.95 0)
+			(at 198.3233 107.95 0)
 			(effects
 				(font
@@
 		)
 	)
-	(global_label "FCU_USB_OTG_FS_DM"
+	(global_label "FCU_USB_OTG_FS_D-"
 		(shape input)
 		(at 175.26 115.57 0)
@@
 		)
 		(property "Intersheetrefs" "${INTERSHEET_REFS}"
-			(at 198.2023 115.57 0)
-			(effects
-				(font
+			(at 198.3233 115.57 0)
+			(effects
+				(font
