File: Hardware/aircraft.kicad_pcb (KiCad board)
At the start: 4 copper layers, 100 x 50 mm, 192 parts, among them J1 Conn_01x02_Pin, J10 Conn_01x06, J12 Conn_02x05_Odd_Even, J13 Conn_01x02, J14 USB_B_Micro, J15 Conn_02x05_Odd_Even, J16 USB_B_Micro, J17 USB_B_Micro, J18 USB_B_Micro, J19 U.FL-R-SMT-1_80_, J2 DM3AT-SF-PEJM5, J3 Conn_01x04, J4 Conn_01x04, J5 Conn_01x10, J6 Conn_02x10_Odd_Even, J7 Conn_01x04, J8 Conn_01x04, J9 Conn_02x06_Odd_Even, SW1 SW_SPDT, SW2 SW_Push_Dual, SW3 SW_SPDT, SW4 SW_Push_Dual, U1 MIC26903YJL-TR, U10 BMP390, U11 W25N01GVZEIG_TR, U12 STM32F405RGTx, U13 W25N01GVZEIG_TR, U14 24CW1280T-I/OT, U15 PCA9685PW_118, U16 CH330N, U17 CH330N, U2 LD39200PU33R, U3 INA226, U4 STM32F405RGTx, U5 IST8310, U6 NEO-M8N, U7 BMI088, U8 TMP100, U9 24CW1280T-I/OT, Y1 25MHz, Y2 25MHz

Commit message: hardware: better layout, no power supply and sensors
Parts:
- C25, R15, R16, R17, R18: moved to B.Cu
- moved C13 114.1 mm to (177.7, 76.7), turned to 90 degrees
- moved C19 110.0 mm to (176.2, 76.2), turned to 180 degrees
- moved C12 107.8 mm to (174.1, 88.8)
- moved R13 107.5 mm to (179.1, 83.3), turned to 90 degrees
- moved C22 107.2 mm to (174.6, 87.3), turned to 90 degrees
- moved R12 106.5 mm to (179.1, 85.3), turned to -90 degrees
- moved C17 106.4 mm to (166.2, 72.5)
- moved R9 103.4 mm to (177.6, 86.8), turned to 180 degrees
- moved R17 103.3 mm to (178.5, 82.3), turned to 90 degrees
- moved R18 102.9 mm to (177.5, 82.3), turned to 90 degrees
- moved C16 101.9 mm to (163.5, 76.2)
- moved R14 101.1 mm to (177.6, 81.8), turned to 180 degrees
- moved R11 99.0 mm to (167.8, 73.0), turned to 90 degrees
- moved C21 98.8 mm to (166.9, 89.2), turned to 180 degrees
- moved C20 98.6 mm to (166.9, 88.2), turned to 180 degrees
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Connections:
- net FCU_USB_OTG_FS_DM renamed FCU_USB_OTG_FS_D-
- net FCU_USB_OTG_FS_DP renamed FCU_USB_OTG_FS_D+
